File: NFCAccessController.brd (EAGLE design)
At the start: 153.7 x 67.9 mm, 141 parts, among them IC1 LD1117S33, IC2 APX811-44UG-7, IC3 W5100SQFP80, IC4 ATmega328P, IC5 MC34063, IC6 HEF4050B, IC7 PN532, J1 POE, J2 Solenoid, J3 Serial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

Commit message: foo
Parts:
- R28: value 1k -> 10k
Changed lines of the file:
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@@
 <element name="R34" library="freetronics-master-v1" package="0603" value="10k" x="34.925" y="71.755"/>
 <element name="LED10" library="freetronics-master-v1" package="LED-0603" value="SD act" x="59.055" y="78.74"/>
-<element name="R28" library="freetronics-master-v1" package="0603" value="1k" x="32.385" y="66.04"/>
+<element name="R28" library="freetronics-master-v1" package="0603" value="10k" x="32.385" y="66.04"/>
 <element name="R29" library="freetronics-master-v1" package="0603" value="10k" x="57.785" y="74.93"/>
 <element name="S$1" library="SparkFun" package="OSHW-LOGO-S" value="OSHW-LOGOS" x="13.335" y="-3.81"/>

Commit message: foo
Connections:
- removed net N$69: J1.1, U1.P$10
- net +12V: now also J1.2
- net GND: now also U1.P$10
- net N$68: now also J1.1; no longer J1.2
Changed lines of the file:
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@@
 <contactref element="C29" pad="2"/>
 <contactref element="C34" pad="2"/>
+<contactref element="U1" pad="P$10"/>
 <wire x1="83.947" y1="72.39" x2="84.582" y2="74.295" width="0" layer="19" extent="1-1"/>
 <wire x1="85.217" y1="69.215" x2="83.947" y2="72.39" width="0" layer="19" extent="1-1"/>
@@
 <wire x1="28.17" y1="23.985" x2="29.42" y2="22.735" width="0" layer="19" extent="1-1"/>
 <wire x1="54.09" y1="16.57" x2="54.09" y2="14.17" width="0" layer="19" extent="1-1"/>
+<wire x1="74.295" y1="19.685" x2="77.595" y2="21.715" width="0" layer="19" extent="1-1"/>
 <wire x1="57.09" y1="19.57" x2="54.09" y2="16.57" width="0" layer="19" extent="1-1"/>
 <wire x1="60.69" y1="19.57" x2="57.09" y2="19.57" width="0" layer="19" extent="1-1"/>
@@
 <wire x1="41.402" y1="73.025" x2="38.1" y2="69.3166" width="0" layer="19" extent="1-1"/>
 <wire x1="41.402" y1="75.565" x2="41.402" y2="73.025" width="0" layer="19" extent="1-1"/>
+<wire x1="47.752" y1="71.755" x2="41.402" y2="73.025" width="0" layer="19" extent="1-1"/>
+<wire x1="50.165" y1="68.707" x2="47.752" y2="71.755" width="0" layer="19" extent="1-1"/>
 <wire x1="47.625" y1="80.01" x2="41.402" y2="75.565" width="0" layer="19" extent="1-1"/>
 <wire x1="50.165" y1="80.01" x2="47.625" y2="80.01" width="0" layer="19" extent="1-1"/>
@@
 <wire x1="32.893" y1="74.93" x2="38.1" y2="69.3166" width="0" layer="19" extent="1-1"/>
 <wire x1="31.75" y1="75.4634" x2="32.893" y2="74.93" width="0" layer="19" extent="1-1"/>
-<wire x1="50.165" y1="68.707" x2="41.402" y2="73.025" width="0" layer="19" extent="1-1"/>
-<wire x1="47.752" y1="71.755" x2="0.198" y2="26.29" width="0" layer="19" extent="1-1"/>
 </signal>
 <signal name="N$1">
@@
 <wire x1="11.43" y1="44.45" x2="11.43" y2="14.605" width="0.8128" layer="16"/>
 <contactref element="D1" pad="1"/>
+<contactref element="J1" pad="2"/>
 <wire x1="80.01" y1="56.515" x2="67.43" y2="74.295" width="0" layer="19" extent="1-1"/>
 <wire x1="76.454" y1="45.085" x2="80.01" y2="56.515" width="0" layer="19" extent="1-1"/>
-<wire x1="15.24" y1="50.165" x2="67.43" y2="74.295" width="0" layer="19" extent="1-1"/>
+<wire x1="26.035" y1="76.835" x2="67.43" y2="74.295" width="0" layer="19" extent="1-1"/>
+<wire x1="15.24" y1="50.165" x2="26.035" y2="76.835" width="0" layer="19" extent="1-1"/>
 </signal>
 <signal name="N$22">
@@
 <signal name="N$68">
 <contactref element="U1" pad="P$9"/>
-<contactref element="J1" pad="2"/>
-<wire x1="71.755" y1="18.415" x2="26.035" y2="76.835" width="0" layer="19" extent="1-1"/>
-</signal>
-<signal name="N$69">
-<contactref element="U1" pad="P$10"/>
 <contactref element="J1" pad="1"/>
-<wire x1="74.295" y1="19.685" x2="23.495" y2="76.835" width="0" layer="19" extent="1-1"/>
+<wire x1="71.755" y1="18.415" x2="23.495" y2="76.835" width="0" layer="19" extent="1-1"/>
 </signal>
 <signal name="1V8_OUT">
