File: NFCAccessController.sch (EAGLE design)
At the start: 137 parts, among them IC1 LD1117S33, IC2 APX811-44UG-7, IC3 W5100SQFP80, IC4 ATmega328P, IC5 MC34063, IC6 HEF4050B, IC7 PN532, J1 POE, J2 Solenoid, J3 Serial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

Commit message: foo
Parts:
- R28: value 1k -> 10k
Other:
- note added: "32-TQFP"
- note added: "887-1421-1-ND"
- note removed: "Q1: 887-1421-1-ND"
- moved on the sheet: C1, C16, C2, C20, C21, C22, C23, IC1, IC4, J3, J5, LED7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

Commit message: foo
Connections:
- removed net N$69: J1.1, U1.V-
- net +12V: now also J1.2
- net GND: now also U1.V-
- net N$68: now also J1.1; no longer J1.2
Other:
- moved on the sheet: J1
Changed lines of the file:
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@@
 <setting verticaltext="up"/>
 </settings>
-<grid distance="0.1" unitdist="inch" unit="inch" style="lines" multiple="1" display="yes" altdistance="0.01" altunitdist="inch" altunit="inch"/>
+<grid distance="0.1" unitdist="inch" unit="inch" style="lines" multiple="1" display="yes" altdistance="0.005" altunitdist="inch" altunit="inch"/>
 <layers>
 <layer number="1" name="Top" color="4" fill="1" visible="no" active="no"/>
@@
 <part name="FRAME1" library="frames" deviceset="A3L-LOC" device="" value="Frame"/>
 <part name="FRAME2" library="frames" deviceset="A3L-LOC" device="" value="Frame"/>
+<part name="P+2" library="supply1" deviceset="+12V" device=""/>
 </parts>
 <sheets>
@@
 <attribute name="VALUE" x="297.18" y="231.14" size="1.27" layer="96"/>
 </instance>
-<instance part="IC1" gate="G$1" x="132.08" y="481.33" smashed="yes">
-<attribute name="NAME" x="126.238" y="487.68" size="1.27" layer="95" ratio="10"/>
-<attribute name="VALUE" x="126.238" y="485.648" size="1.27" layer="96" ratio="10"/>
+<instance part="IC1" gate="G$1" x="131.953" y="481.33" smashed="yes">
+<attribute name="NAME" x="126.111" y="487.68" size="1.27" layer="95" ratio="10"/>
+<attribute name="VALUE" x="126.111" y="485.648" size="1.27" layer="96" ratio="10"/>
 </instance>
 <instance part="J4" gate="G$1" x="231.14" y="175.26" smashed="yes">
@@
 <attribute name="VALUE" x="127" y="416.56" size="1.27" layer="96"/>
 </instance>
-<instance part="J1" gate="G$1" x="109.22" y="436.88" smashed="yes" rot="R90">
-<attribute name="NAME" x="114.3" y="434.34" size="1.27" layer="95"/>
-<attribute name="VALUE" x="114.3" y="431.8" size="1.27" layer="96"/>
+<instance part="J1" gate="G$1" x="111.76" y="441.96" smashed="yes" rot="R90">
+<attribute name="NAME" x="116.84" y="439.42" size="1.27" layer="95"/>
+<attribute name="VALUE" x="116.84" y="436.88" size="1.27" layer="96"/>
 </instance>
 <instance part="U$75" gate="G$1" x="175.26" y="467.36"/>
@@
 <instance part="FRAME1" gate="G$1" x="0" y="0"/>
 <instance part="FRAME2" gate="G$1" x="0" y="264.16"/>
+<instance part="P+2" gate="1" x="127" y="431.8" smashed="yes" rot="R270">
+<attribute name="VALUE" x="127" y="434.34" size="1.27" layer="96"/>
+</instance>
 </instances>
 <busses>
@@
 <pinref part="IC1" gate="G$1" pin="GND"/>
 <pinref part="U$65" gate="G$1" pin="GND"/>
-<wire x1="132.08" y1="469.9" x2="132.207" y2="474.98" width="0.1524" layer="91"/>
+<wire x1="132.08" y1="469.9" x2="132.08" y2="474.98" width="0.1524" layer="91"/>
 </segment>
 <segment>
@@
 </segment>
 <segment>
-<wire x1="101.6" y1="424.18" x2="114.3" y2="424.18" width="0.1524" layer="91"/>
+<wire x1="101.6" y1="424.18" x2="106.68" y2="424.18" width="0.1524" layer="91"/>
+<wire x1="106.68" y1="424.18" x2="114.3" y2="424.18" width="0.1524" layer="91"/>
 <wire x1="101.6" y1="426.72" x2="114.3" y2="426.72" width="0.1524" layer="91"/>
 <pinref part="U1" gate="G$1" pin="GND1"/>
@@
 <wire x1="114.3" y1="424.18" x2="114.3" y2="426.72" width="0.1524" layer="91"/>
 <junction x="114.3" y="424.18"/>
+<wire x1="101.6" y1="406.4" x2="106.68" y2="406.4" width="0.1524" layer="91"/>
+<wire x1="106.68" y1="406.4" x2="106.68" y2="424.18" width="0.1524" layer="91"/>
+<pinref part="U1" gate="G$1" pin="V-"/>
+<junction x="106.68" y="424.18"/>
 </segment>
 <segment>
@@
 <segment>
 <pinref part="IC1" gate="G$1" pin="VOUT"/>
-<wire x1="141.097" y1="482.6" x2="144.78" y2="482.6" width="0.1524" layer="91"/>
+<wire x1="140.97" y1="482.6" x2="144.78" y2="482.6" width="0.1524" layer="91"/>
 <wire x1="144.78" y1="480.06" x2="144.78" y2="482.6" width="0.1524" layer="91"/>
 <pinref part="U$57" gate="G$1" pin="+3V3"/>
@@
 <pinref part="C1" gate="G$1" pin="1"/>
 <pinref part="IC1" gate="G$1" pin="VIN"/>
-<wire x1="123.317" y1="482.6" x2="119.38" y2="482.6" width="0.1524" layer="91"/>
+<wire x1="123.19" y1="482.6" x2="119.38" y2="482.6" width="0.1524" layer="91"/>
 <wire x1="119.38" y1="482.6" x2="119.38" y2="485.14" width="0.1524" layer="91"/>
 <junction x="119.38" y="482.6"/>
@@
 <junction x="243.84" y="243.84"/>
 </segment>
+<segment>
+<pinref part="P+2" gate="1" pin="+12V"/>
+<pinref part="J1" gate="G$1" pin="2"/>
+<wire x1="124.46" y1="431.8" x2="111.76" y2="431.8" width="0.1524" layer="91"/>
+<wire x1="111.76" y1="431.8" x2="111.76" y2="439.42" width="0.1524" layer="91"/>
+</segment>
 </net>
 <net name="N$22" class="0">
@@
 <segment>
 <wire x1="101.6" y1="403.86" x2="109.22" y2="403.86" width="0.1524" layer="91"/>
-<wire x1="109.22" y1="403.86" x2="109.22" y2="434.34" width="0.1524" layer="91"/>
 <pinref part="U1" gate="G$1" pin="V+"/>
-<pinref part="J1" gate="G$1" pin="2"/>
-</segment>
-</net>
-<net name="N$69" class="0">
-<segment>
-<wire x1="101.6" y1="406.4" x2="106.68" y2="406.4" width="0.1524" layer="91"/>
-<wire x1="106.68" y1="406.4" x2="106.68" y2="434.34" width="0.1524" layer="91"/>
-<pinref part="U1" gate="G$1" pin="V-"/>
 <pinref part="J1" gate="G$1" pin="1"/>
-</segment>
-</net>
+<wire x1="109.22" y1="403.86" x2="109.22" y2="439.42" width="0.1524" layer="91"/>
+</segment>
+</net>
